Commit message: Finished milestone 2 hexapod robot

File: body.urdf (robot description, URDF)
Before this commit: robot robot, 3 links, 2 joints
Links:
- added link BackLowerLeg, mass 1; collision box size=0.2 0.2 1; visual box size=0.2 0.2 1
- added link FrontLowerLeg, mass 1; collision box size=0.2 0.2 1; visual box size=0.2 0.2 1
- added link LeftLeg, mass 1; collision box size=1 0.2 0.2; visual box size=1 0.2 0.2
- added link LeftLowerLeg, mass 1; collision box size=0.2 0.2 1; visual box size=0.2 0.2 1
- added link MiddleLeftLeg, mass 1; collision box size=1 0.2 0.2; visual box size=1 0.2 0.2
- added link MiddleLeftLowerLeg, mass 1; collision box size=0.2 0.2 1; visual box size=0.2 0.2 1
- added link MiddleRightLeg, mass 1; collision box size=1 0.2 0.2; visual box size=1 0.2 0.2
- added link MiddleRightLowerLeg, mass 1; collision box size=0.2 0.2 1; visual box size=0.2 0.2 1
- added link RightLeg, mass 1; collision box size=1 0.2 0.2; visual box size=1 0.2 0.2
- added link RightLowerLeg, mass 1; collision box size=0.2 0.2 1; visual box size=0.2 0.2 1
- link BackLeg: geometry collision box size=0.2 1 0.2; visual box size=0.2 1 0.2
- link FrontLeg: geometry collision box size=0.2 1 0.2; visual box size=0.2 1 0.2
Joints:
- added joint BackLeg_BackLowerLeg: type revolute, parent BackLeg, child BackLowerLeg, origin xyz=0 -1.0 0 rpy=0 0 0, axis 1 0 0, limit lower=-3.14159 upper=3.14159 effort=0.0 velocity=0.0
- added joint FrontLeg_FrontLowerLeg: type revolute, parent FrontLeg, child FrontLowerLeg, origin xyz=0 1.0 0 rpy=0 0 0, axis 1 0 0, limit lower=-3.14159 upper=3.14159 effort=0.0 velocity=0.0
- added joint LeftLeg_LeftLowerLeg: type revolute, parent LeftLeg, child LeftLowerLeg, origin xyz=-1.0 0 0 rpy=0 0 0, axis 0 1 0, limit lower=-3.14159 upper=3.14159 effort=0.0 velocity=0.0
- added joint MiddleLeftLeg_MiddleLeftLowerLeg: type revolute, parent MiddleLeftLeg, child MiddleLeftLowerLeg, origin xyz=-1.0 0 0 rpy=0 0 0, axis 0 1 0, limit lower=-3.14159 upper=3.14159 effort=0.0 velocity=0.0
- added joint MiddleRightLeg_MiddleRightLowerLeg: type revolute, parent MiddleRightLeg, child MiddleRightLowerLeg, origin xyz=1.0 0 0 rpy=0 0 0, axis 0 1 0, limit lower=-3.14159 upper=3.14159 effort=0.0 velocity=0.0
- added joint RightLeg_RightLowerLeg: type revolute, parent RightLeg, child RightLowerLeg, origin xyz=1.0 0 0 rpy=0 0 0, axis 0 1 0, limit lower=-3.14159 upper=3.14159 effort=0.0 velocity=0.0
- added joint Torso_LeftLeg: type revolute, parent Torso, child LeftLeg, origin xyz=-0.5 0 1 rpy=0 0 0, axis 0 1 0, limit lower=-3.14159 upper=3.14159 effort=0.0 velocity=0.0
- added joint Torso_MiddleLeftLeg: type revolute, parent Torso, child MiddleLeftLeg, origin xyz=-0.5 -0.5 1 rpy=0 0 0, axis 0 1 0, limit lower=-3.14159 upper=3.14159 effort=0.0 velocity=0.0
- added joint Torso_MiddleRightLeg: type revolute, parent Torso, child MiddleRightLeg, origin xyz=0.5 0.5 1 rpy=0 0 0, axis 0 1 0, limit lower=-3.14159 upper=3.14159 effort=0.0 velocity=0.0
- added joint Torso_RightLeg: type revolute, parent Torso, child RightLeg, origin xyz=0.5 0 1 rpy=0 0 0, axis 0 1 0, limit lower=-3.14159 upper=3.14159 effort=0.0 velocity=0.0
- joint Torso_BackLeg: axis 0 1 0 -> 1 0 0; origin xyz=1.0 0 1.0 rpy=0 0 0 -> xyz=0 -0.5 1.0 rpy=0 0 0
- joint Torso_FrontLeg: axis 0 1 0 -> 1 0 0; origin xyz=2.0 0 1.0 rpy=0 0 0 -> xyz=0 0.5 1.0 rpy=0 0 0

Commit message: Collected quadruped comparison data for milestone 3

File: body.urdf (robot description, URDF)
Before this commit: robot robot, 13 links, 12 joints
Links:
- removed link MiddleLeftLeg
- removed link MiddleLeftLowerLeg
- removed link MiddleRightLeg
- removed link MiddleRightLowerLeg
Joints:
- removed joint MiddleLeftLeg_MiddleLeftLowerLeg
- removed joint MiddleRightLeg_MiddleRightLowerLeg
- removed joint Torso_MiddleLeftLeg
- removed joint Torso_MiddleRightLeg

Commit message: Fixed hexapod leg positioning

File: body.urdf (robot description, URDF)
Before this commit: robot robot, 13 links, 12 joints
Joints:
- joint Torso_MiddleLeftLeg: origin xyz=-0.5 -0.5 1 rpy=0 0 0 -> xyz=-0.5 -0.25 1 rpy=0 0 0
- joint Torso_MiddleRightLeg: origin xyz=0.5 0.5 1 rpy=0 0 0 -> xyz=0.5 0.25 1 rpy=0 0 0
